Commit message: + commenti

File: src/bluerov2_description/urdf/hydrodynamics.xacro (robot description, xacro)
@@ -1,21 +1,24 @@
 <?xml version="1.0"?>
+<!-- Descrizione delle dinamiche idrodinamiche del BlueROV2 per Ignition Gazebo -->
 <xacro>
 <gazebo>
+    <!-- Plugin di Ignition Gazebo che applica forze idrodinamiche (massa aggiunta, smorzamenti) -->
     <plugin filename="ignition-gazebo-hydrodynamics-system" name="ignition::gazebo::systems::Hydrodynamics">
+<!--     Densità del fluido (acqua). Può essere passato come argomento da bluerov2.xacro -->
 <!--     <density>${density}</density> -->
-    <!-- Ignition notations from Handbook of Marine Craft, Fossen, 2011 -->
+    <!-- Convenzioni/Notazioni secondo il "Handbook of Marine Craft" di Fossen (2011) usate da Ignition -->
+    <!-- Link del veicolo a cui applicare le forze idrodinamiche -->
     <link_name>${ns}/base_link</link_name>
-    <!-- BlueROV2 heavy values from "6-DoF Modelling and Control of a Remotely Operated Vehicle"
-        Wu, Master thesis, Flinder University, 2018  -->
-    <!-- Negative diagonal values of added mass matrix [Fossen (6.38)] -->
-    <xDotU>-5.5</xDotU>
-    <yDotV>-12.7</yDotV>
-    <zDotW>-14.57</zDotW>
-    <kDotP>-0.12</kDotP>
-    <mDotQ>-0.12</mDotQ>
-    <nDotR>-0.12</nDotR>
-    <!-- From "Numerical Modelling and Experimental Testing of the Hydrodynamic Characteristics
-        for an Open-Frame Remotely Operated Vehicle",  Li et al, Marine Science and Engineering, 2020         -->
-    <!-- Negative linear damping [Fossen (6.62)] -->
+    <!-- Valori del BlueROV2 (versione heavy) da "6-DoF Modelling and Control of a Remotely Operated Vehicle",
+         Wu, Master thesis, Flinders University, 2018 -->
+    <!-- Valori diagonali negativi della matrice di massa aggiunta [Fossen (6.38)] -->
+    <xDotU>-5.5</xDotU>   <!-- Massa aggiunta in surge -->
+    <yDotV>-12.7</yDotV>  <!-- Massa aggiunta in sway -->
+    <zDotW>-14.57</zDotW> <!-- Massa aggiunta in heave -->
+    <kDotP>-0.12</kDotP>  <!-- Massa aggiunta in roll -->
+    <mDotQ>-0.12</mDotQ>  <!-- Massa aggiunta in pitch -->
+    <nDotR>-0.12</nDotR>  <!-- Massa aggiunta in yaw -->
+    <!-- Valori alternativi dalla letteratura (Li et al., 2020) - smorzamenti lineari/quadratici -->
+    <!-- Smorzamento lineare negativo [Fossen (6.62)] -->
 <!--    <xU>-1.31</xU>
     <yV>-9.14</yV>
@@ -24,5 +27,5 @@
     <mQ>-0.</mQ>
     <nR>-0.</nR>-->
-    <!-- Negative quadratic damping [Fossen (6.62)] -->
+    <!-- Smorzamento quadratico negativo [Fossen (6.62)] -->
 <!--      <xUabsU>-33.800000000000004</xUabsU>
       <yVabsV>-54.26875</yVabsV>
@@ -31,14 +34,14 @@
       <mQabsQ>-40.0</mQabsQ>
       <nRabsR>-40.0</nRabsR>-->
-    <!-- BlueROV2 values from "Model Predictive Control for the BlueROV2",
-        Emil Már Einarsson, Andris Lipenitis, Master thesis, 2020  -->
-    <!-- Negative linear damping -->
-    <xU>-25.15</xU>
-    <yV>-7.364</yV>
-    <zW>-17.955</zW>
-    <kP>-10.888</kP>
-    <mQ>-20.761</mQ>
-    <nR>-3.744</nR>
-    <!-- Negative quadratic damping -->
+    <!-- Valori del BlueROV2 da "Model Predictive Control for the BlueROV2",
+         Emil Már Einarsson, Andris Lipenitis, Master thesis, 2020 -->
+    <!-- Smorzamenti lineari negativi (proporzionali alla velocità) -->
+    <xU>-25.15</xU>   <!-- Damping in surge -->
+    <yV>-7.364</yV>   <!-- Damping in sway -->
+    <zW>-17.955</zW>  <!-- Damping in heave -->
+    <kP>-10.888</kP>  <!-- Damping in roll -->
+    <mQ>-20.761</mQ>  <!-- Damping in pitch -->
+    <nR>-3.744</nR>   <!-- Damping in yaw -->
+    <!-- Smorzamenti quadratici negativi (proporzionali al quadrato della velocità) -->
     <xUabsU>-17.77</xUabsU>
     <yVabsV>-125.9</yVabsV>

File: src/bluerov2_description/urdf/sensors.xacro (robot description, xacro)
@@ -1,8 +1,13 @@
 <?xml version="1.0"?>
+<!-- Sensori del BlueROV2: IMU, camera con tilt, sonar Ping360 e controller -->
 <robot xmlns:xacro="http://www.ros.org/wiki/xacro">
+<!-- Offset X della camera rispetto al base_link e valore di PI -->
 <xacro:property name="x_camera" value="0.02"/>
 <xacro:property name="PI" value="3.1415927"/>
+<!-- Macro per creare un link IMU e un sensore IMU in Gazebo -->
 <xacro:macro name="imu" params="name *origin">
+    <!-- Link del sensore IMU -->
     <link name="${ns}/${name}"/>
+    <!-- Configurazione del sensore IMU in Gazebo -->
     <gazebo reference="${ns}/${name}">
     <sensor name="${name}_imu" type="imu">
@@ -13,4 +18,5 @@
             <gz_frame_id>${ns}/${name}</gz_frame_id>
       <imu>
+        <!-- Rumore gaussiano su velocità angolare (x,y,z) -->
         <angular_velocity>
           <x>
@@ -48,4 +54,5 @@
           </z>
         </angular_velocity>
+        <!-- Rumore gaussiano su accelerazione lineare (x,y,z) -->
         <linear_acceleration>
           <x>
@@ -83,4 +90,5 @@
           </z>
         </linear_acceleration>
+        <!-- Riferimento di orientazione ENU (East-North-Up) -->
         <orientation_reference_frame>
           <localization>ENU</localization>
@@ -89,4 +97,5 @@
         </sensor>
       </gazebo>
+     <!-- Giunto fisso per collegare l'IMU al base_link del veicolo -->
      <joint name="${name}" type="fixed">
         <xacro:insert_block name="origin"/>
@@ -95,14 +104,17 @@
     </joint>
 </xacro:macro>
+<!-- Istanziazione IMU tipo MPU -->
 <xacro:imu name="mpu">
-    <origin xyz="0.1 0 0" rpy="0 0 ${-PI/2}"/>
+  <origin xyz="0.1 0 0" rpy="0 0 ${-PI/2}"/>
 </xacro:imu>
+<!-- Istanziazione IMU tipo LSM -->
 <xacro:imu name="lsm">
-    <origin xyz="0.1 0 0" rpy="0 0 ${-PI/2}"/>
+  <origin xyz="0.1 0 0" rpy="0 0 ${-PI/2}"/>
 </xacro:imu>
-  <!-- Pressure Sensor  -->
+  <!-- Sensore di pressione (barometro) - opzionale/commentato -->
 <!--  <xacro:default_pressure parent_link="${ns}/base_link" sensor_name="baro">
     <origin xyz="0 0 0" rpy="0 0 0"/>
   </xacro:default_pressure>-->
+  <!-- Link della camera con inerzia semplificata -->
   <link name="${ns}/camera">
     <inertial>
@@ -117,4 +129,5 @@
     </inertial>
  </link>
+<!-- Giunto di tilt della camera (asse Y) -->
 <joint name="tilt" type="revolute">
     <parent link="${ns}/base_link"/>
@@ -125,5 +138,7 @@
     <dynamics damping="0.8"/>
 </joint>
+<!-- Link del frame ottico della camera (convenzione ROS) -->
 <link name="${ns}/camera_optical"/>
+<!-- Giunto fisso tra camera e frame ottico -->
 <joint name="camera_optical" type="fixed">
     <parent link="${ns}/camera"/>
@@ -131,4 +146,5 @@
     <origin rpy="${-PI/2} 0 ${-PI/2}"/>
 </joint>
+<!-- Link del sonar Ping360 -->
 <link name="${ns}/sonar">
     <visual>
@@ -140,4 +156,5 @@
     </visual>
 </link>
+<!-- Giunto fisso per montare il sonar sul base_link -->
 <joint name="sonar" type="fixed">
     <parent link="${ns}/base_link"/>
@@ -145,4 +162,5 @@
     <origin xyz="0.135 0.108 0.118"/>
 </joint>
+<!-- Sensore sonar basato su GPU Ray -->
 <gazebo reference="${ns}/sonar">
   <sensor type="gpu_ray" name="ping360_sonar">
@@ -179,4 +197,5 @@
   </sensor>
 </gazebo>
+<!-- Controller PID di posizione per il giunto tilt della camera -->
 <gazebo>
     <plugin filename="ignition-gazebo-joint-position-controller-system" name="ignition::gazebo::systems::JointPositionController">
@@ -189,4 +208,5 @@
     </plugin>
 </gazebo>
+ <!-- Sensore camera RGB con frame ottico e parametri immagine -->
  <gazebo reference="${ns}/camera">
   <sensor name="camera" type="camera">

File: src/bluerov2_description/urdf/thrusters.xacro (robot description, xacro)
@@ -1,9 +1,12 @@
 <?xml version="1.0"?>
+<!-- Definizione dei propulsori (thruster) del BlueROV2: link, joint e plugin -->
 <robot xmlns:xacro="http://www.ros.org/wiki/xacro">
+  <!-- Mesh delle eliche: cw (orario) e ccw (antiorario) -->
   <xacro:property name="prop_mesh_cw" value="package://bluerov2_description/meshes/bluerov2_propcw.dae"/>
   <xacro:property name="prop_mesh_ccw" value="package://bluerov2_description/meshes/bluerov2_propccw.dae"/>
+  <!-- Raggio e lunghezza della geometria dell'elica -->
   <xacro:property name="prop_r" value="0.05"/>
   <xacro:property name="prop_l" value="0.035"/>
-  <!--  Thruster macro: joint + link + plugin -->
+  <!-- Macro del thruster: crea link, joint e plugin per un propulsore -->
   <xacro:macro name="thruster" params="thruster_id *origin">
     <link name="${ns}/thruster${thruster_id}">
@@ -25,7 +28,9 @@
       </collision>-->
      <inertial>
-     <!-- thruster axis is X -->
+     <!-- L'asse del thruster è X; posizioniamo l'origine al centro geometrico -->
       <origin xyz="${prop_l/2} 0 0" rpy="0 0 0" />
+      <!-- Massa dell'elica (prop_mass definita in bluerov2.xacro) -->
       <mass value="${prop_mass}" />
+      <!-- Inerzia dell'elica approssimata come cilindro sottile -->
       <inertia  izz="${prop_mass*prop_r*prop_r / 4  + prop_mass*prop_l*prop_l / 12}" ixy="0.0"  ixz="0.0"
                 iyy="${prop_mass*prop_r*prop_r / 4  + prop_mass*prop_l*prop_l / 12}" iyz="0.0"
@@ -33,5 +38,5 @@
     </inertial>
     </link>
-    <!-- Joint between thruster link and vehicle base link -->
+    <!-- Giunto tra il link del thruster e il base_link del veicolo -->
     <joint name="thruster${thruster_id}" type="continuous">
       <xacro:insert_block name="origin" />
@@ -46,5 +51,5 @@
       <limits effort="-1" velocity="-1"/>
     </joint>
-    <!-- ignition topic is /model/{ns}/joint/{joint_name}/cmd_pos -->
+    <!-- Plugin di Ignition per controllare il thruster (comandi su topic ROS/Ignition) -->
 <!--    <xacro:if value="$(arg simulation)"> -->
     <gazebo>
@@ -55,9 +60,14 @@
             <joint_name>thruster${thruster_id}</joint_name>
             <topic>thruster${thruster_id}/cmd</topic>
+            <!-- Coefficiente di spinta del propulsore (relazione forza-comando) -->
             <thrust_coefficient>0.011</thrust_coefficient>
+            <!-- Densità del fluido (acqua), passata da bluerov2.xacro -->
             <fluid_density>${density}</fluid_density>
+            <!-- Diametro dell'elica -->
             <propeller_diameter>${2*prop_r}</propeller_diameter>
+            <!-- Controllo in velocità (true) invece che angolare -->
             <velocity_control>true</velocity_control>
             <use_angvel_cmd>false</use_angvel_cmd>
+            <!-- Limiti del comando di spinta -->
             <max_thrust_cmd>40</max_thrust_cmd>
             <min_thrust_cmd>-40</min_thrust_cmd>
@@ -66,5 +76,5 @@
 <!--  </xacro:if> -->
 </xacro:macro>
-  <!-- all 6 thrusters -->
+  <!-- Istanziazione di tutti e 6 i thruster con posizioni e orientazioni -->
   <xacro:thruster thruster_id="1">
     <origin xyz="0.1355 -0.1 -0.0725" rpy="0 0 0.7853981634"/>
